Commit message: working gui button

File: car/install/car_description/share/car_description/urdf/newcar.xacro (robot description, xacro)
@@ -1,189 +1 @@
-<?xml version="1.0"?>
-<robot xmlns:xacro="http://www.ros.org/wiki/xacro" name="newcar">
-  <!-- ================= BASE LINK ================= -->
-  <link name="base_link">
-    <visual>
-      <origin xyz="0 0 0" rpy="0 0 0"/>
-      <geometry>
-        <mesh filename="package://car_description/meshes/panther/base.dae"/>
-      </geometry>
-    </visual>
-    <collision>
-      <origin xyz="0 0 0" rpy="0 0 0"/>
-      <geometry>
-        <mesh filename="package://car_description/meshes/panther/base_collision.stl"/>
-      </geometry>
-    </collision>
-    <inertial>
-      <origin xyz="0 0 0.1"/>
-      <mass value="15.0"/>
-      <inertia ixx="0.5" ixy="0" ixz="0"
-               iyy="0.8" iyz="0"
-               izz="1.0"/>
-    </inertial>
-  </link>
-  <!-- ================= REAR LEFT WHEEL ================= -->
-  <link name="rear_left_wheel_link">
-    <visual>
-      <geometry>
-        <mesh filename="package://car_description/meshes/WH05/rl_wheel.dae"/>
-      </geometry>
-    </visual>
-    <collision>
-      <origin rpy="1.5708 0 0"/>
-      <geometry>
-        <cylinder radius="0.12" length="0.08"/>
-      </geometry>
-    </collision>
-    <inertial>
-      <mass value="2.0"/>
-      <inertia ixx="0.015" iyy="0.015" izz="0.015"
-               ixy="0" ixz="0" iyz="0"/>
-    </inertial>
-  </link>
-  <!-- ================= REAR RIGHT WHEEL ================= -->
-  <link name="rear_right_wheel_link">
-    <visual>
-      <geometry>
-        <mesh filename="package://car_description/meshes/WH05/rr_wheel.dae"/>
-      </geometry>
-    </visual>
-    <collision>
-      <origin rpy="1.5708 0 0"/>
-      <geometry>
-        <cylinder radius="0.12" length="0.08"/>
-      </geometry>
-    </collision>
-    <inertial>
-      <mass value="2.0"/>
-      <inertia ixx="0.015" iyy="0.015" izz="0.015"
-               ixy="0" ixz="0" iyz="0"/>
-    </inertial>
-  </link>
-  <!-- ================= FRONT CASTER (CLUSTER) WHEEL ================= -->
-  <link name="front_caster_wheel_link">
-    <visual>
-      <geometry>
-        <sphere radius="0.06"/>
-      </geometry>
-    </visual>
-    <collision>
-      <geometry>
-        <sphere radius="0.06"/>
-      </geometry>
-    </collision>
-    <inertial>
-      <mass value="0.5"/>
-      <inertia ixx="0.0005" iyy="0.0005" izz="0.0005"
-               ixy="0" ixz="0" iyz="0"/>
-    </inertial>
-  </link>
-  <!-- ================= LIDAR ================= -->
-  <link name="lidar_link">
-    <visual>
-      <geometry>
-        <mesh filename="package://car_description/meshes/WH05/G1.STL"/>
-      </geometry>
-    </visual>
-    <collision>
-      <geometry>
-        <cylinder radius="0.05" length="0.07"/>
-      </geometry>
-    </collision>
-    <inertial>
-      <mass value="0.5"/>
-      <inertia ixx="0.001" iyy="0.001" izz="0.001"
-               ixy="0" ixz="0" iyz="0"/>
-    </inertial>
-  </link>
-  <!-- ================= JOINTS ================= -->
-  <joint name="rear_left_wheel_joint" type="continuous">
-    <parent link="base_link"/>
-    <child link="rear_left_wheel_link"/>
-    <origin xyz="-0.23 0.32 0.01"/>
-    <axis xyz="0 1 0"/>
-  </joint>
-  <joint name="rear_right_wheel_joint" type="continuous">
-    <parent link="base_link"/>
-    <child link="rear_right_wheel_link"/>
-    <origin xyz="-0.23 -0.32 0.01"/>
-    <axis xyz="0 1 0"/>
-  </joint>
-  <!-- Free rotating caster -->
-  <joint name="front_caster_joint" type="continuous">
-    <parent link="base_link"/>
-    <child link="front_caster_wheel_link"/>
-    <origin xyz="0.10 0 -0.05"/>
-    <axis xyz="0 0 1"/>
-    <dynamics damping="0.05"/>
-  </joint>
-  <!-- Lidar joint -->
-  <joint name="lidar_joint" type="fixed">
-    <parent link="base_link"/>
-    <child link="lidar_link"/>
-    <origin xyz="0.12 0 0.20"/>
-  </joint>
-  <!-- ================= GAZEBO DIFF DRIVE ================= -->
-  <gazebo>
-    <plugin name="diff_drive" filename="libgazebo_ros_diff_drive.so">
-      <left_joint>rear_left_wheel_joint</left_joint>
-      <right_joint>rear_right_wheel_joint</right_joint>
-      <wheel_separation>0.64</wheel_separation>
-      <wheel_diameter>0.24</wheel_diameter>
-      <max_wheel_torque>200</max_wheel_torque>
-      <max_wheel_acceleration>10.0</max_wheel_acceleration>
-      <robot_base_frame>base_link</robot_base_frame>
-      <publish_odom>true</publish_odom>
-      <publish_odom_tf>true</publish_odom_tf>
-    </plugin>
-  </gazebo>
-  <!-- ================= LIDAR GAZEBO SENSOR ================= -->
-<gazebo reference="lidar_link">
-  <sensor type="ray" name="lidar_sensor">
-    <pose>0 0 0 0 0 0</pose>
-    <visualize>true</visualize>
-    <update_rate>10</update_rate>
-    <ray>
-      <scan>
-        <horizontal>
-          <samples>360</samples>
-          <resolution>1</resolution>
-          <min_angle>-3.14159</min_angle>
-          <max_angle>3.14159</max_angle>
-        </horizontal>
-      </scan>
-      <range>
-        <min>0.1</min>
-        <max>12.0</max>
-        <resolution>0.01</resolution>
-      </range>
-      <noise>
-        <type>gaussian</type>
-        <mean>0.0</mean>
-        <stddev>0.01</stddev>
-      </noise>
-    </ray>
-    <!-- ROS2 Gazebo plugin -->
-    <plugin name="gazebo_ros_lidar" filename="libgazebo_ros_ray_sensor.so">
-      <ros>
-        <remapping>~/out:=/scan</remapping>
-      </ros>
-      <frame_name>lidar_link</frame_name>
-      <output_type>sensor_msgs/LaserScan</output_type>
-    </plugin>
-  </sensor>
-</gazebo>
-  <!-- ================= FRICTION TUNING ================= -->
-  <gazebo reference="rear_left_wheel_link">
-    <mu1>1.2</mu1>
-    <mu2>1.2</mu2>
-  </gazebo>
-  <gazebo reference="rear_right_wheel_link">
-    <mu1>1.2</mu1>
-    <mu2>1.2</mu2>
-  </gazebo>
-  <gazebo reference="front_caster_wheel_link">
-    <mu1>0.05</mu1>
-    <mu2>0.05</mu2>
-  </gazebo>
-</robot>
+/home/samay/AVG/car/src/car_description/urdf/newcar.xacro

Commit message: added cargo platform

File: car/install/car_description/share/car_description/urdf/newcar.xacro (robot description, xacro)
@@ -1 +1,468 @@
-/home/samay/AVG/car/src/car_description/urdf/newcar.xacro
+<?xml version="1.0"?>
+<robot xmlns:xacro="http://www.ros.org/wiki/xacro" name="newcar">
+  <!-- ================= BASE LINK ================= -->
+  <link name="base_link">
+    <visual>
+      <origin xyz="0 0 0" rpy="0 0 0"/>
+      <geometry>
+        <mesh filename="package://car_description/meshes/panther/base.dae"/>
+      </geometry>
+    </visual>
+    <collision>
+      <origin xyz="0 0 0" rpy="0 0 0"/>
+      <geometry>
+        <mesh filename="package://car_description/meshes/panther/base_collision.stl"/>
+      </geometry>
+    </collision>
+    <inertial>
+      <origin xyz="0 0 0.1"/>
+      <mass value="15.0"/>
+      <inertia ixx="0.5" ixy="0" ixz="0"
+               iyy="0.8" iyz="0"
+               izz="1.0"/>
+    </inertial>
+  </link>
+  <!-- ================= PILLAR 1 (Front Left) ================= -->
+  <link name="pillar_front_left_link">
+    <visual>
+      <geometry>
+        <cylinder radius="0.02" length="1.25"/>
+      </geometry>
+      <material name="pillar_color">
+        <color rgba="0.2 0.2 0.2 1.0"/>
+      </material>
+    </visual>
+    <collision>
+      <geometry>
+        <cylinder radius="0.02" length="1.25"/>
+      </geometry>
+    </collision>
+    <inertial>
+      <mass value="2.5"/>
+      <inertia ixx="0.325" ixy="0" ixz="0"
+               iyy="0.325" iyz="0"
+               izz="0.0001"/>
+    </inertial>
+  </link>
+  <!-- ================= PILLAR 2 (Front Right) ================= -->
+  <link name="pillar_front_right_link">
+    <visual>
+      <geometry>
+        <cylinder radius="0.02" length="1.25"/>
+      </geometry>
+      <material name="pillar_color">
+        <color rgba="0.2 0.2 0.2 1.0"/>
+      </material>
+    </visual>
+    <collision>
+      <geometry>
+        <cylinder radius="0.02" length="1.25"/>
+      </geometry>
+    </collision>
+    <inertial>
+      <mass value="2.5"/>
+      <inertia ixx="0.325" ixy="0" ixz="0"
+               iyy="0.325" iyz="0"
+               izz="0.0001"/>
+    </inertial>
+  </link>
+  <!-- ================= PILLAR 3 (Rear Left) ================= -->
+  <link name="pillar_rear_left_link">
+    <visual>
+      <geometry>
+        <cylinder radius="0.02" length="1.25"/>
+      </geometry>
+      <material name="pillar_color">
+        <color rgba="0.2 0.2 0.2 1.0"/>
+      </material>
+    </visual>
+    <collision>
+      <geometry>
+        <cylinder radius="0.02" length="1.25"/>
+      </geometry>
+    </collision>
+    <inertial>
+      <mass value="2.5"/>
+      <inertia ixx="0.325" ixy="0" ixz="0"
+               iyy="0.325" iyz="0"
+               izz="0.0001"/>
+    </inertial>
+  </link>
+  <!-- ================= PILLAR 4 (Rear Right) ================= -->
+  <link name="pillar_rear_right_link">
+    <visual>
+      <geometry>
+        <cylinder radius="0.02" length="1.25"/>
+      </geometry>
+      <material name="pillar_color">
+        <color rgba="0.2 0.2 0.2 1.0"/>
+      </material>
+    </visual>
+    <collision>
+      <geometry>
+        <cylinder radius="0.02" length="1.25"/>
+      </geometry>
+    </collision>
+    <inertial>
+      <mass value="2.5"/>
+      <inertia ixx="0.325" ixy="0" ixz="0"
+               iyy="0.325" iyz="0"
+               izz="0.0001"/>
+    </inertial>
+  </link>
+  <!-- ================= CARGO PLATFORM ================= -->
+  <link name="cargo_platform_link">
+    <visual>
+      <geometry>
+        <box size="0.40 0.50 0.02"/>
+      </geometry>
+      <material name="platform_color">
+        <color rgba="0.6 0.4 0.2 1.0"/>
+      </material>
+    </visual>
+    <collision>
+      <geometry>
+        <box size="0.40 0.50 0.02"/>
+      </geometry>
+    </collision>
+    <inertial>
+      <mass value="1.5"/>
+      <inertia ixx="0.032" ixy="0" ixz="0"
+               iyy="0.021" iyz="0"
+               izz="0.051"/>
+    </inertial>
+  </link>
+  <!-- ================= CARGO BOUNDARY WALLS ================= -->
+  <!-- Front boundary -->
+  <link name="cargo_boundary_front">
+    <visual>
+      <geometry>
+        <box size="0.02 0.50 0.08"/>
+      </geometry>
+      <material name="boundary_color">
+        <color rgba="0.4 0.3 0.1 1.0"/>
+      </material>
+    </visual>
+    <collision>
+      <geometry>
+        <box size="0.02 0.50 0.08"/>
+      </geometry>
+    </collision>
+    <inertial>
+      <mass value="0.2"/>
+      <inertia ixx="0.0007" ixy="0" ixz="0"
+               iyy="0.0001" iyz="0"
+               izz="0.0007"/>
+    </inertial>
+  </link>
+  <!-- Rear boundary -->
+  <link name="cargo_boundary_rear">
+    <visual>
+      <geometry>
+        <box size="0.02 0.50 0.08"/>
+      </geometry>
+      <material name="boundary_color">
+        <color rgba="0.4 0.3 0.1 1.0"/>
+      </material>
+    </visual>
+    <collision>
+      <geometry>
+        <box size="0.02 0.50 0.08"/>
+      </geometry>
+    </collision>
+    <inertial>
+      <mass value="0.2"/>
+      <inertia ixx="0.0007" ixy="0" ixz="0"
+               iyy="0.0001" iyz="0"
+               izz="0.0007"/>
+    </inertial>
+  </link>
+  <!-- Left boundary -->
+  <link name="cargo_boundary_left">
+    <visual>
+      <geometry>
+        <box size="0.40 0.02 0.08"/>
+      </geometry>
+      <material name="boundary_color">
+        <color rgba="0.4 0.3 0.1 1.0"/>
+      </material>
+    </visual>
+    <collision>
+      <geometry>
+        <box size="0.40 0.02 0.08"/>
+      </geometry>
+    </collision>
+    <inertial>
+      <mass value="0.2"/>
+      <inertia ixx="0.0001" ixy="0" ixz="0"
+               iyy="0.0007" iyz="0"
+               izz="0.0007"/>
+    </inertial>
+  </link>
+  <!-- Right boundary -->
+  <link name="cargo_boundary_right">
+    <visual>
+      <geometry>
+        <box size="0.40 0.02 0.08"/>
+      </geometry>
+      <material name="boundary_color">
+        <color rgba="0.4 0.3 0.1 1.0"/>
+      </material>
+    </visual>
+    <collision>
+      <geometry>
+        <box size="0.40 0.02 0.08"/>
+      </geometry>
+    </collision>
+    <inertial>
+      <mass value="0.2"/>
+      <inertia ixx="0.0001" ixy="0" ixz="0"
+               iyy="0.0007" iyz="0"
+               izz="0.0007"/>
+    </inertial>
+  </link>
+  <!-- ================= REAR LEFT WHEEL ================= -->
+  <link name="rear_left_wheel_link">
+    <visual>
+      <geometry>
+        <mesh filename="package://car_description/meshes/WH05/rl_wheel.dae"/>
+      </geometry>
+    </visual>
+    <collision>
+      <origin rpy="1.5708 0 0"/>
+      <geometry>
+        <cylinder radius="0.12" length="0.08"/>
+      </geometry>
+    </collision>
+    <inertial>
+      <mass value="2.0"/>
+      <inertia ixx="0.015" iyy="0.015" izz="0.015"
+               ixy="0" ixz="0" iyz="0"/>
+    </inertial>
+  </link>
+  <!-- ================= REAR RIGHT WHEEL ================= -->
+  <link name="rear_right_wheel_link">
+    <visual>
+      <geometry>
+        <mesh filename="package://car_description/meshes/WH05/rr_wheel.dae"/>
+      </geometry>
+    </visual>
+    <collision>
+      <origin rpy="1.5708 0 0"/>
+      <geometry>
+        <cylinder radius="0.12" length="0.08"/>
+      </geometry>
+    </collision>
+    <inertial>
+      <mass value="2.0"/>
+      <inertia ixx="0.015" iyy="0.015" izz="0.015"
+               ixy="0" ixz="0" iyz="0"/>
+    </inertial>
+  </link>
+  <!-- ================= FRONT CASTER (CLUSTER) WHEEL ================= -->
+  <link name="front_caster_wheel_link">
+    <visual>
+      <geometry>
+        <sphere radius="0.06"/>
+      </geometry>
+    </visual>
+    <collision>
+      <geometry>
+        <sphere radius="0.06"/>
+      </geometry>
+    </collision>
+    <inertial>
+      <mass value="0.5"/>
+      <inertia ixx="0.0005" iyy="0.0005" izz="0.0005"
+               ixy="0" ixz="0" iyz="0"/>
+    </inertial>
+  </link>
+  <!-- ================= LIDAR ================= -->
+  <link name="lidar_link">
+    <visual>
+      <geometry>
+        <mesh filename="package://car_description/meshes/WH05/G1.STL"/>
+      </geometry>
+    </visual>
+    <collision>
+      <geometry>
+        <cylinder radius="0.05" length="0.07"/>
+      </geometry>
+    </collision>
+    <inertial>
+      <mass value="0.5"/>
+      <inertia ixx="0.001" iyy="0.001" izz="0.001"
+               ixy="0" ixz="0" iyz="0"/>
+    </inertial>
+  </link>
+  <!-- ================= JOINTS ================= -->
+  <!-- Pillar joints - fixed to base at four corners -->
+  <joint name="pillar_front_left_joint" type="fixed">
+    <parent link="base_link"/>
+    <child link="pillar_front_left_link"/>
+    <origin xyz="0.15 0.20 0.8" rpy="0 0 0"/>
+  </joint>
+  <joint name="pillar_front_right_joint" type="fixed">
+    <parent link="base_link"/>
+    <child link="pillar_front_right_link"/>
+    <origin xyz="0.15 -0.20 0.8" rpy="0 0 0"/>
+  </joint>
+  <joint name="pillar_rear_left_joint" type="fixed">
+    <parent link="base_link"/>
+    <child link="pillar_rear_left_link"/>
+    <origin xyz="-0.15 0.20 0.8" rpy="0 0 0"/>
+  </joint>
+  <joint name="pillar_rear_right_joint" type="fixed">
+    <parent link="base_link"/>
+    <child link="pillar_rear_right_link"/>
+    <origin xyz="-0.15 -0.20 0.8" rpy="0 0 0"/>
+  </joint>
+  <!-- Cargo platform joint - sits on top of pillars -->
+  <joint name="cargo_platform_joint" type="fixed">
+    <parent link="base_link"/>
+    <child link="cargo_platform_link"/>
+    <origin xyz="0 0 1.4" rpy="0 0 0"/>
+  </joint>
+  <!-- Cargo boundary joints -->
+  <joint name="cargo_boundary_front_joint" type="fixed">
+    <parent link="cargo_platform_link"/>
+    <child link="cargo_boundary_front"/>
+    <origin xyz="0.21 0 0.05" rpy="0 0 0"/>
+  </joint>
+  <joint name="cargo_boundary_rear_joint" type="fixed">
+    <parent link="cargo_platform_link"/>
+    <child link="cargo_boundary_rear"/>
+    <origin xyz="-0.21 0 0.05" rpy="0 0 0"/>
+  </joint>
+  <joint name="cargo_boundary_left_joint" type="fixed">
+    <parent link="cargo_platform_link"/>
+    <child link="cargo_boundary_left"/>
+    <origin xyz="0 0.26 0.05" rpy="0 0 0"/>
+  </joint>
+  <joint name="cargo_boundary_right_joint" type="fixed">
+    <parent link="cargo_platform_link"/>
+    <child link="cargo_boundary_right"/>
+    <origin xyz="0 -0.26 0.05" rpy="0 0 0"/>
+  </joint>
+  <joint name="rear_left_wheel_joint" type="continuous">
+    <parent link="base_link"/>
+    <child link="rear_left_wheel_link"/>
+    <origin xyz="-0.23 0.32 0.01"/>
+    <axis xyz="0 1 0"/>
+  </joint>
+  <joint name="rear_right_wheel_joint" type="continuous">
+    <parent link="base_link"/>
+    <child link="rear_right_wheel_link"/>
+    <origin xyz="-0.23 -0.32 0.01"/>
+    <axis xyz="0 1 0"/>
+  </joint>
+  <!-- Free rotating caster -->
+  <joint name="front_caster_joint" type="continuous">
+    <parent link="base_link"/>
+    <child link="front_caster_wheel_link"/>
+    <origin xyz="0.10 0 -0.05"/>
+    <axis xyz="0 0 1"/>
+    <dynamics damping="0.05"/>
+  </joint>
+  <!-- Lidar joint -->
+  <joint name="lidar_joint" type="fixed">
+    <parent link="base_link"/>
+    <child link="lidar_link"/>
+    <origin xyz="0.12 0 0.20"/>
+  </joint>
+  <!-- ================= GAZEBO DIFF DRIVE ================= -->
+  <gazebo>
+    <plugin name="diff_drive" filename="libgazebo_ros_diff_drive.so">
+      <left_joint>rear_left_wheel_joint</left_joint>
+      <right_joint>rear_right_wheel_joint</right_joint>
+      <wheel_separation>0.64</wheel_separation>
+      <wheel_diameter>0.24</wheel_diameter>
+      <max_wheel_torque>200</max_wheel_torque>
+      <max_wheel_acceleration>10.0</max_wheel_acceleration>
+      <robot_base_frame>base_link</robot_base_frame>
+      <publish_odom>true</publish_odom>
+      <publish_odom_tf>true</publish_odom_tf>
+    </plugin>
+  </gazebo>
+  <!-- ================= LIDAR GAZEBO SENSOR ================= -->
+  <gazebo reference="lidar_link">
+    <sensor type="ray" name="lidar_sensor">
+      <pose>0 0 0 0 0 0</pose>
+      <visualize>true</visualize>
+      <update_rate>10</update_rate>
+      <ray>
+        <scan>
+          <horizontal>
+            <samples>360</samples>
+            <resolution>1</resolution>
+            <min_angle>-3.14159</min_angle>
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